Commit message: Fix sensor conflicts, upgrade to gazebo11, but tf_tree still has some errors

File: livox/livox_laser_simulation/urdf/livox_avia.xacro (robot description, xacro)
@@ -88,5 +88,5 @@
     <xacro:Livox_Mid_gazebo_sensor name="${name}" visualize="${visualize}"/>
   </xacro:macro>
-    <xacro:Livox_AVIA name="livox" visualize="false" />
+    <xacro:Livox_AVIA name="livox"/>
   <xacro:include filename="$(find livox_laser_simulation)/urdf/standardrobots_oasis300.xacro"/>
   <xacro:link_oasis name="oasis"/>

File: scout_gazebo/urdf/base1.xacro (robot description, xacro)
@@ -1,5 +1,4 @@
 <?xml version="1.0"?>
-<robot name="scout_v2"  xmlns:xacro="http://ros.org/wiki/xacro">
-    <xacro:arg name="robot_namespace" default="/" />
+<robot name="scout_v2"  xmlns:xacro="http://ros.org/wiki/xacro">W
     <!-- 属性封装 -->
     <xacro:property name="M_PI" value="3.14159"/>
@@ -16,18 +15,25 @@
     <xacro:arg name="organize_cloud" default="true"/>
     <xacro:property name="organize_cloud" value="$(arg organize_cloud)" />
-    <material name="black">
-        <color rgba="0.0 0.0 0.0 1.0" />
+    <!-- Defining the colors used in this robot -->
+    <material name="Black">
+        <color rgba="0 0 0 1"/>
     </material>
-    <!-- 底盘的轮子 -->
-    <xacro:include filename="$(find scout_gazebo)/urdf/scout_wheel_type1.xacro" />
-    <xacro:include filename="$(find scout_gazebo)/urdf/scout_wheel_type2.xacro" />
+    <material name="White">
+        <color rgba="1 1 1 1"/>
+    </material>
+    <material name="Blue">
+        <color rgba="0 0 1 1"/>
+    </material>
+    <material name="Red">
+        <color rgba="1 0 0 1"/>
+    </material>
     <xacro:include filename="$(find scout_gazebo)/urdf/inertial.xacro" />
-    <!-- <xacro:include filename="$(find scout_gazebo)/urdf/camera.xacro" /> -->
-    <!-- <xacro:include filename="$(find scout_gazebo)/urdf/sensor_camera.xacro" /> -->
-    <!-- D435i RGB-D相机相关 -->
-    <xacro:include filename="$(find realsense_ros_gazebo)/xacro/depthcam.xacro"/>
-    <xacro:realsense_d435 sensor_name="camera" parent_link="base_link" rate="30.0">
-    <origin rpy="0 0 0" xyz="0 0 0.3"/>
-    </xacro:realsense_d435>
+	<!-- inertial matrix -->
+	<xacro:macro name="inertial_matrix" params="mass">
+        <inertial>
+            <mass value="${mass}" />
+            <inertia ixx="1.0" ixy="0.0" ixz="0.0" iyy="0.5" iyz="0.0" izz="1.0" />
+        </inertial>
+    </xacro:macro>
     <!-- VLP16 激光雷达 -->
     <!--xacro:include filename="$(find scout_gazebo)/urdf/laser_support.xacro" />
@@ -40,5 +46,5 @@
     <xacro:include filename="$(find scout_gazebo)/urdf/livox_avia.xacro"/>
     <xacro:Livox_AVIA name="livox" visualize="true" parent="support"/>
-    <joint name="livox_base_joint" type="fixed">
+   <joint name="livox_base_joint" type="fixed">
         <parent link="support"/>
         <child link="livox_base"/>
@@ -46,5 +52,10 @@
                 xyz="0.04 0 ${support_length/2}"/>
     </joint>
-    <!-- IMU 模块 -->
+    <!-- D435i RGB-D相机相关 -->
+ <!--   <xacro:include filename="$(find realsense_ros_gazebo)/xacro/depthcam1.xacro"/>
+    <xacro:realsense_d435 sensor_name="camera" parent_link="base_link" rate="30.0">
+    <origin rpy="0 0 0" xyz="0 0 0.3"/>
+    </xacro:realsense_d435>-->
+   <!-- IMU 模块 -->
     <xacro:include filename="$(find scout_gazebo)/urdf/imu.xacro"/>
     <xacro:imu sensor_name="imu" parent_link="base_link">
@@ -53,4 +64,5 @@
     <!-- 机器人导航控制模块 -->
     <xacro:include filename="$(find scout_gazebo)/urdf/move.xacro" />
+    <!-- base_link -->
     <!-- Base link  底盘 -->
     <link name="base_link">
@@ -69,4 +81,7 @@
         </collision>
     </link>
+    <gazebo reference="base_link">
+        <material>Gazebo/White</material>
+    </gazebo>
     <link name="base_footprint"/>
     <joint name="base_footprint_joint" type="fixed">
@@ -75,5 +90,5 @@
         <child link="base_footprint" />
     </joint>
-    <link name="inertial_link">
+        <link name="inertial_link">
         <inertial>
             <mass value="40" />
@@ -87,18 +102,3 @@
         <child link="inertial_link" />
     </joint>
-    <!-- 宏  Scout wheel macros -->
-    <!-- wheel labeled from 0 to 3, conter-clockwise, starting from front right wheel -->
-    <!-- motor 1 and 2 (left side) are mechanically installed in a reversed direction -->
-    <xacro:scout_wheel_type1 wheel_prefix="front_right">
-        <origin xyz="${wheelbase/2} ${-track/2} ${wheel_vertical_offset}" rpy="3.14 0 0" />
-    </xacro:scout_wheel_type1>
-    <xacro:scout_wheel_type2 wheel_prefix="front_left">
-        <origin xyz="${wheelbase/2} ${track/2} ${wheel_vertical_offset}" rpy="0 0 0" />
-    </xacro:scout_wheel_type2>
-    <xacro:scout_wheel_type1 wheel_prefix="rear_left">
-        <origin xyz="${-wheelbase/2} ${track/2} ${wheel_vertical_offset}" rpy="0 0 0" />
-    </xacro:scout_wheel_type1>
-    <xacro:scout_wheel_type2 wheel_prefix="rear_right">
-        <origin xyz="${-wheelbase/2} ${-track/2} ${wheel_vertical_offset}" rpy="3.14 0 0" />
-    </xacro:scout_wheel_type2>
 </robot>

File: scout_gazebo/urdf/laser_support.xacro (robot description, xacro)
@@ -25,4 +25,6 @@
         </collision>
         <xacro:cylinder_inertial_matrix m="${support_m}" r="${support_radius}" h="${support_length}" />
+        <kinematic>1</kinematic>
+		<gravity>9.8</gravity>
     </link>
     <joint name="support2base_link" type="fixed">

File: scout_gazebo/urdf/livox_avia.xacro (robot description, xacro)
@@ -1,4 +1,4 @@
 <?xml version="1.0"?>
-<robot xmlns:xacro="http://ros.org/wiki/xacro">
+<robot name="livox_a"  xmlns:xacro="http://wiki.ros.org/xacro">
   <xacro:property name="M_PI" value="3.14159"/>
   <xacro:property name="laser_min_range" value="0.1"/>
@@ -12,11 +12,11 @@
     <inertial>
       <mass value="0.1"/>
-    <inertia ixx="0.01" ixy="0" ixz="0"
-          iyy="0.01" iyz="0"
-          izz="0.01"/>
+      <origin xyz="0.0 0.0 0.0" />
+     <inertia ixx="0.01" ixy="0" ixz="0" iyy="0.01" iyz="0" izz="0.01"/>
     </inertial>
   </xacro:macro>
   <xacro:macro name="Livox_Mid_gazebo_sensor" params="visualize:=True update_rate:=10 resolution:=0.002 noise_mean:=0.0 noise_stddev:=0.01 name:=livox">
     <gazebo reference="${name}">
+        <gravity>1</gravity>
       <sensor type="ray" name="laser_${name}">
         <pose>0 0 0 0 0 0</pose>
@@ -59,6 +59,12 @@
       </sensor>
     </gazebo>
+<!--    <joint name="${name}_to_laser_${name}_joint" type="fixed">
+      <parent link="${name}"/>
+      <child link="laser_${name}"/>
+      <origin rpy="0 0 0" xyz="0.0 0.0 0.0"/>
+    </joint>
+    -->
   </xacro:macro>
-  <xacro:macro name="Livox_AVIA" params="visualize:=True name:=livox">
+  <xacro:macro name="Livox_AVIA" params="visualize:=True name:=livox parent:=base_link">
     <link name="${name}_base">
       <xacro:null_inertial/>
@@ -87,7 +93,13 @@
     </joint>
     <xacro:Livox_Mid_gazebo_sensor name="${name}" visualize="${visualize}"/>
+    <!--  not elegent solution for sensor's tf error    -->
+    <!--<joint name="${name}_to_${name}_sensor_joint" type="fixed">
+      <parent link="${name}"/>
+      <child link="laser_${name}"/>
+      <origin rpy="0 0 0" xyz="0.0 0.0 0.0"/>
+    </joint>   -->
   </xacro:macro>
-    <!--xacro:Livox_AVIA name="livox" visualize="false" /-->
-  <!--xacro:include filename="$(find livox_laser_simulation)/urdf/standardrobots_oasis300.xacro"/>
-  <xacro:link_oasis name="oasis"/-->
+<!--    <xacro:Livox_AVIA name="livox" visualize="true" />-->
+<!--  <xacro:include filename="$(find livox_laser_simulation)/urdf/standardrobots_oasis300.xacro"/>
+  <xacro:link_oasis name="oasis"/>-->
 </robot>
