Commit message: Adapt livox plugin to gazebo11 and fix tf_tree problem

File: livox/livox_laser_simulation_gz11/urdf/livox_avia.xacro (robot description, xacro)
@@ -3,9 +3,8 @@
   <xacro:property name="M_PI" value="3.14159"/>
   <xacro:property name="laser_min_range" value="0.1"/>
-  <xacro:property name="laser_max_range" value="40.0"/>
+  <xacro:property name="laser_max_range" value="200.0"/>
   <xacro:property name="horizontal_fov" value="70.4"/>
   <xacro:property name="vertical_fov" value="77.2"/>
   <xacro:property name="ros_topic" value="scan"/>
-  <!-- <xacro:property name="samples" value="24000"/> -->
   <xacro:property name="samples" value="24000"/>
   <xacro:property name="downsample" value="1"/>

File: livox/livox_laser_simulation_gz11/urdf/livox_horizon.xacro (robot description, xacro)
@@ -3,14 +3,13 @@
   <xacro:property name="M_PI" value="3.14159"/>
   <xacro:property name="laser_min_range" value="0.1"/>
-  <xacro:property name="laser_max_range" value="40.0"/>
-  <xacro:property name="horizontal_fov" value="70.4"/>
-  <xacro:property name="vertical_fov" value="77.2"/>
-  <xacro:property name="ros_topic" value="scan"/>
-  <!-- <xacro:property name="samples" value="24000"/> -->
+  <xacro:property name="laser_max_range" value="200.0"/>
+  <xacro:property name="horizontal_fov" value="81.7"/>
+  <xacro:property name="vertical_fov" value="25.1"/>
+  <xacro:property name="ros_topic" value="livox/lidar"/>
   <xacro:property name="samples" value="24000"/>
-  <xacro:property name="downsample" value="1"/>
-  <xacro:property name="csv_file_name" value="package://livox_laser_simulation/scan_mode/avia.csv"/>
+  <xacro:property name="publish_pointcloud_type" value="0"/>
+  <xacro:property name="csv_file_name" value="package://livox_laser_simulation/scan_mode/horizon.csv"/>
   <xacro:include filename="$(find livox_laser_simulation)/urdf/livox_gazebo_sensor.xacro"/>
-  <xacro:macro name="Livox_Avia" params="visualize:=True name:=livox publish_pointcloud_type:=0">
+  <xacro:macro name="Livox_Horizon" params="visualize:=True name:=livox publish_pointcloud_type:=0 ros_topic:=livox/lidar downsample:=1">
     <link name="${name}_base">
       <xacro:null_inertial/>
@@ -23,9 +22,9 @@
       </visual>
       <collision>
-          <origin xyz="0 0 0" rpy="0 0 0" />
-          <geometry>
-          <mesh filename="package://livox_laser_simulation/meshes/livox_mid40.dae">
-          </mesh>
-          </geometry>
+		  <origin xyz="0.00 0 0.00" rpy="0 0 0" />
+      <geometry>
+        <mesh filename="package://livox_laser_simulation/meshes/livox_mid40.dae">
+		    </mesh>
+      </geometry>
       </collision>
     </link>
@@ -38,4 +37,10 @@
       <origin rpy="0 0 0" xyz="0.0 0.0 0.0"/>
     </joint>
+    <link name="${name}_imu_link"/>
+    <joint name="imu_link_joint" type="fixed">
+      <parent link="${name}"/>
+      <child link="${name}_imu_link"/>
+      <origin rpy="0 0 0" xyz="-0.05512 -0.02226 0.0297"/>
+    </joint>
     <xacro:Livox_gazebo_sensor name="${name}" visualize="${visualize}" publish_pointcloud_type="${publish_pointcloud_type}"/>
   </xacro:macro>

File: livox/livox_laser_simulation_gz11/urdf/livox_mid40.xacro (robot description, xacro)
@@ -3,14 +3,14 @@
   <xacro:property name="M_PI" value="3.14159"/>
   <xacro:property name="laser_min_range" value="0.1"/>
-  <xacro:property name="laser_max_range" value="40.0"/>
-  <xacro:property name="horizontal_fov" value="70.4"/>
-  <xacro:property name="vertical_fov" value="77.2"/>
+  <xacro:property name="laser_max_range" value="200.0"/>
+  <xacro:property name="horizontal_fov" value="38.4"/>
+  <xacro:property name="vertical_fov" value="38.4"/>
   <xacro:property name="ros_topic" value="scan"/>
-  <!-- <xacro:property name="samples" value="24000"/> -->
-  <xacro:property name="samples" value="24000"/>
+  <xacro:property name="samples" value="10000"/>
   <xacro:property name="downsample" value="1"/>
-  <xacro:property name="csv_file_name" value="package://livox_laser_simulation/scan_mode/avia.csv"/>
+  <xacro:property name="publish_pointcloud_type" value="0"/>
+  <xacro:property name="csv_file_name" value="package://livox_laser_simulation/scan_mode/mid40.csv"/>
   <xacro:include filename="$(find livox_laser_simulation)/urdf/livox_gazebo_sensor.xacro"/>
-  <xacro:macro name="Livox_Avia" params="visualize:=True name:=livox publish_pointcloud_type:=0">
+  <xacro:macro name="Livox_Mid40" params="visualize:=True name:=livox publish_pointcloud_type:=1 ros_topic:=scan">
     <link name="${name}_base">
       <xacro:null_inertial/>
@@ -38,5 +38,5 @@
       <origin rpy="0 0 0" xyz="0.0 0.0 0.0"/>
     </joint>
-    <xacro:Livox_gazebo_sensor name="${name}" visualize="${visualize}" publish_pointcloud_type="${publish_pointcloud_type}"/>
+    <xacro:Livox_gazebo_sensor name="${name}" visualize="${visualize}"/>
   </xacro:macro>
 </robot>

File: livox/livox_laser_simulation_gz11/urdf/livox_mid70.xacro (robot description, xacro)
@@ -3,14 +3,13 @@
   <xacro:property name="M_PI" value="3.14159"/>
   <xacro:property name="laser_min_range" value="0.1"/>
-  <xacro:property name="laser_max_range" value="40.0"/>
+  <xacro:property name="laser_max_range" value="200.0"/>
   <xacro:property name="horizontal_fov" value="70.4"/>
-  <xacro:property name="vertical_fov" value="77.2"/>
+  <xacro:property name="vertical_fov" value="70.4"/>
   <xacro:property name="ros_topic" value="scan"/>
-  <!-- <xacro:property name="samples" value="24000"/> -->
-  <xacro:property name="samples" value="24000"/>
+  <xacro:property name="samples" value="10000"/>
   <xacro:property name="downsample" value="1"/>
-  <xacro:property name="csv_file_name" value="package://livox_laser_simulation/scan_mode/avia.csv"/>
+  <xacro:property name="csv_file_name" value="package://livox_laser_simulation/scan_mode/mid70.csv"/>
   <xacro:include filename="$(find livox_laser_simulation)/urdf/livox_gazebo_sensor.xacro"/>
-  <xacro:macro name="Livox_Avia" params="visualize:=True name:=livox publish_pointcloud_type:=0">
+  <xacro:macro name="Livox_Mid70" params="visualize:=True name:=livox publish_pointcloud_type:=0">
     <link name="${name}_base">
       <xacro:null_inertial/>

File: livox/livox_laser_simulation_gz11/urdf/livox_tele.xacro (robot description, xacro)
@@ -3,14 +3,13 @@
   <xacro:property name="M_PI" value="3.14159"/>
   <xacro:property name="laser_min_range" value="0.1"/>
-  <xacro:property name="laser_max_range" value="40.0"/>
-  <xacro:property name="horizontal_fov" value="70.4"/>
-  <xacro:property name="vertical_fov" value="77.2"/>
+  <xacro:property name="laser_max_range" value="200.0"/>
+  <xacro:property name="horizontal_fov" value="14.5"/>
+  <xacro:property name="vertical_fov" value="16.1"/>
   <xacro:property name="ros_topic" value="scan"/>
-  <!-- <xacro:property name="samples" value="24000"/> -->
   <xacro:property name="samples" value="24000"/>
   <xacro:property name="downsample" value="1"/>
-  <xacro:property name="csv_file_name" value="package://livox_laser_simulation/scan_mode/avia.csv"/>
+  <xacro:property name="csv_file_name" value="package://livox_laser_simulation/scan_mode/mid70.csv"/>
   <xacro:include filename="$(find livox_laser_simulation)/urdf/livox_gazebo_sensor.xacro"/>
-  <xacro:macro name="Livox_Avia" params="visualize:=True name:=livox publish_pointcloud_type:=0">
+  <xacro:macro name="Livox_Tele" params="visualize:=True name:=livox publish_pointcloud_type:=0">
     <link name="${name}_base">
       <xacro:null_inertial/>

File: scout_gazebo/urdf/base.xacro (robot description, xacro)
@@ -38,6 +38,10 @@
     <!-- livox AVIA激光雷达 -->
     <xacro:include filename="$(find scout_gazebo)/urdf/laser_support.xacro" />
-    <xacro:include filename="$(find scout_gazebo)/urdf/livox_avia.xacro"/>
-    <xacro:Livox_AVIA name="livox" visualize="true" parent="support"/>
+  <xacro:include filename="$(find scout_gazebo)/urdf/livox_avia.xacro"/>
+  <Livox_Avia name="livox" visualize="false" publish_pointcloud_type="0"/>
+    <!-- <xacro:include filename="$(find livox_laser_simulation)/urdf/livox_horizon.xacro"/>
+  <Livox_Horizon name="livox" visualize="true" publish_pointcloud_type="2"/> -->
+<!--    <xacro:include filename="$(find scout_gazebo)/urdf/livox_avia.xacro"/>
+    <xacro:Livox_AVIA name="livox" visualize="true" parent="support"/>-->
     <joint name="livox_base_joint" type="fixed">
         <parent link="support"/>
