Commit message: relocate the cam and livox to avoid shadow

File: scout_gazebo/urdf/base.xacro (robot description, xacro)
@@ -2,4 +2,5 @@
 <robot name="scout_v2"  xmlns:xacro="http://ros.org/wiki/xacro">
     <xacro:arg name="robot_namespace" default="/" />
+    <xacro:property name="CAM_LASER_X_BIAS" value="0.1"/>
     <!-- 属性封装 -->
     <xacro:property name="M_PI" value="3.14159"/>
@@ -28,5 +29,5 @@
     <xacro:include filename="$(find realsense_ros_gazebo)/xacro/depthcam.xacro"/>
     <xacro:realsense_d435 sensor_name="camera" parent_link="base_link" rate="30.0">
-    <origin rpy="0 0 0" xyz="0 0 0.3"/>
+    <origin rpy="0 0 0" xyz="${CAM_LASER_X_BIAS} 0 0.3"/>
     </xacro:realsense_d435>
     <!-- VLP16 激光雷达 -->
@@ -40,13 +41,15 @@
   <xacro:include filename="$(find scout_gazebo)/urdf/livox_avia.xacro"/>
   <Livox_Avia name="livox" visualize="false" publish_pointcloud_type="0"/>
-    <!-- <xacro:include filename="$(find livox_laser_simulation)/urdf/livox_horizon.xacro"/>
-  <Livox_Horizon name="livox" visualize="true" publish_pointcloud_type="2"/> -->
-<!--    <xacro:include filename="$(find scout_gazebo)/urdf/livox_avia.xacro"/>
-    <xacro:Livox_AVIA name="livox" visualize="true" parent="support"/>-->
-    <joint name="livox_base_joint" type="fixed">
+<!--    <joint name="livox_base_joint" type="fixed">
         <parent link="support"/>
         <child link="livox_base"/>
         <origin rpy="0 0 0"
                 xyz="0.04 0 ${support_length/2}"/>
+    </joint>-->
+    <joint name="livox_base_joint" type="fixed">
+        <parent link="base_link"/>
+        <child link="livox_base"/>
+        <origin rpy="0 0 0"
+                xyz="${CAM_LASER_X_BIAS} 0 0.4"/>
     </joint>
     <!-- IMU 模块 -->

Commit message: set livox pointcloud type

File: scout_gazebo/urdf/base.xacro (robot description, xacro)
@@ -40,5 +40,5 @@
     <xacro:include filename="$(find scout_gazebo)/urdf/laser_support.xacro" />
   <xacro:include filename="$(find scout_gazebo)/urdf/livox_avia.xacro"/>
-  <Livox_Avia name="livox" visualize="false" publish_pointcloud_type="0"/>
+  <Livox_Avia name="livox" visualize="false" publish_pointcloud_type="1"/>
 <!--    <joint name="livox_base_joint" type="fixed">
         <parent link="support"/>

File: scout_gazebo/urdf/livox_avia.xacro (robot description, xacro)
@@ -6,5 +6,5 @@
   <xacro:property name="horizontal_fov" value="70.4"/>
   <xacro:property name="vertical_fov" value="77.2"/>
-  <xacro:property name="ros_topic" value="scan"/>
+  <xacro:property name="ros_topic" value="livox/lidar"/>
   <!-- <xacro:property name="samples" value="24000"/> -->
   <xacro:property name="samples" value="24000"/>
